File: src/hardware/RcEsp32Board/RcEsp32Board.kicad_pcb (KiCad board)
At the start: 2 copper layers, 55 x 45 mm, 63 parts, among them IC2 FT231XS-R, J1 Conn_01x02, J10 Conn_01x04, J2 USB_B_Micro, J3 Conn_01x04, J4 Conn_02x04_Odd_Even, J5 Conn_01x03, J6 Conn_01x04, J7 Conn_02x04_Odd_Even, J8 Conn_01x04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

Commit message: update sch/pcb, add gerber data.
Parts:
- removed LD2: LED, FootPrints:LED_1206_HandSoldering
- removed the REF** at (41.5, 38.6)
- removed the REF** at (29.8, 43.9)
- removed the REF** at (29.9, 38.6)
- removed the REF** at (50.1, 34.6)
- removed the REF** at (32.9, 30.7)
- removed the REF** at (67.7, 21.7)
- removed the REF** at (73.5, 28.4)
- removed the REF** at (67.5, 39.5)
- removed the REF** at (73.3, 39.4)
- removed the REF** at (58.0, 50.9)
- removed the REF** at (38.9, 38.6)
- removed the REF** at (56.7, 55.0)
- removed the REF** at (57.9, 62.9)
- removed the REF** at (44.8, 63.5)
- removed the REF** at (44.7, 59.7)
- removed the REF** at (44.7, 56.9)
- removed the REF** at (34.7, 40.8)
- removed the REF** at (29.9, 40.8)
- removed the REF** at (27.2, 22.5)
- removed the REF** at (34.7, 38.6)
- removed the REF** at (23.7, 33.9)
- removed the REF** at (69.2, 25.4)
- removed the REF** at (21.4, 33.9)
- removed the REF** at (49.9, 25.1)
- removed the REF** at (67.8, 50.8)
- removed the REF** at (65.0, 47.6)
- removed the REF** at (57.9, 56.7)
- added LD1: LED, FootPrints:LED_1206_HandSoldering, F.Cu at (42.2, 59.6)
- added REF**: via, FootPrints:via, F.Cu at (51.6, 46.1)
- added REF**: via, FootPrints:via, F.Cu at (73.8, 50.4)
- added REF**: via, FootPrints:via, F.Cu at (73.3, 39.1)
- added REF**: via, FootPrints:via, F.Cu at (67.5, 39.1)
- added REF**: via, FootPrints:via, F.Cu at (64.9, 47.6)
- added REF**: via, FootPrints:via, F.Cu at (67.7, 51.1)
- added REF**: via, FootPrints:via, F.Cu at (62.9, 51.5)
- added REF**: via, FootPrints:via, F.Cu at (69.1, 59.5)
- added REF**: via, FootPrints:via, F.Cu at (58.1, 63.4)
- added REF**: via, FootPrints:via, F.Cu at (58.1, 56.3)
- added REF**: via, FootPrints:via, F.Cu at (56.3, 56.3)
- added REF**: via, FootPrints:via, F.Cu at (50.0, 36.4)
- added REF**: via, FootPrints:via, F.Cu at (56.3, 54.1)
- added REF**: via, FootPrints:via, F.Cu at (57.2, 50.5)
- added REF**: via, FootPrints:via, F.Cu at (47.8, 50.3)
- added REF**: via, FootPrints:via, F.Cu at (53.7, 54.0)
- added REF**: via, FootPrints:via, F.Cu at (53.7, 56.3)
- added REF**: via, FootPrints:via, F.Cu at (51.2, 56.3)
- added REF**: via, FootPrints:via, F.Cu at (48.0, 56.4)
- added REF**: via, FootPrints:via, F.Cu at (44.5, 56.3)
- added REF**: via, FootPrints:via, F.Cu at (44.6, 63.8)
- added REF**: via, FootPrints:via, F.Cu at (44.5, 62.4)
- added REF**: via, FootPrints:via, F.Cu at (50.0, 33.8)
- added REF**: via, FootPrints:via, F.Cu at (44.5, 59.9)
- added REF**: via, FootPrints:via, F.Cu at (39.5, 59.8)
- added REF**: via, FootPrints:via, F.Cu at (33.5, 62.6)
- added REF**: via, FootPrints:via, F.Cu at (34.1, 59.4)
- added REF**: via, FootPrints:via, F.Cu at (34.1, 55.4)
- added REF**: via, FootPrints:via, F.Cu at (30.3, 46.3)
- added REF**: via, FootPrints:via, F.Cu at (29.8, 44.4)
- added REF**: via, FootPrints:via, F.Cu at (29.8, 43.0)
- added REF**: via, FootPrints:via, F.Cu at (29.8, 41.3)
- added REF**: via, FootPrints:via, F.Cu at (29.8, 39.7)
- added REF**: via, FootPrints:via, F.Cu at (50.0, 27.6)
- added REF**: via, FootPrints:via, F.Cu at (29.8, 38.4)
- added REF**: via, FootPrints:via, F.Cu at (34.0, 39.6)
- added REF**: via, FootPrints:via, F.Cu at (35.3, 39.6)
- added REF**: via, FootPrints:via, F.Cu at (41.5, 39.6)
- added REF**: via, FootPrints:via, F.Cu at (41.5, 38.6)
- added REF**: via, FootPrints:via, F.Cu at (39.0, 38.5)
- added REF**: via, FootPrints:via, F.Cu at (34.0, 38.4)
- added REF**: via, FootPrints:via, F.Cu at (36.4, 32.2)
- added REF**: via, FootPrints:via, F.Cu at (36.4, 30.4)
- added REF**: via, FootPrints:via, F.Cu at (36.4, 28.8)
- added REF**: via, FootPrints:via, F.Cu at (50.0, 25.1)
- added REF**: via, FootPrints:via, F.Cu at (32.1, 31.1)
- added REF**: via, FootPrints:via, F.Cu at (28.8, 29.6)
- added REF**: via, FootPrints:via, F.Cu at (28.8, 26.2)
- added REF**: via, FootPrints:via, F.Cu at (33.1, 25.2)
- added REF**: via, FootPrints:via, F.Cu at (33.1, 22.0)
- added REF**: via, FootPrints:via, F.Cu at (26.3, 23.8)
- added REF**: via, FootPrints:via, F.Cu at (28.1, 21.9)
- added REF**: via, FootPrints:via, F.Cu at (26.3, 21.9)
- added REF**: via, FootPrints:via, F.Cu at (25.8, 33.9)
- added REF**: via, FootPrints:via, F.Cu at (73.7, 26.8)
- added REF**: via, FootPrints:via, F.Cu at (21.7, 33.9)
- added REF**: via, FootPrints:via, F.Cu at (69.4, 25.9)
- added REF**: via, FootPrints:via, F.Cu at (67.9, 21.5)
- added REF**: via, FootPrints:via, F.Cu at (65.1, 31.8)
Routing:
- net GND: track 7.82 -> 12.9 mm
Other:
- rule pad_to_mask_clearance: 0.2 -> 0.05

Commit message: update
Parts:
- removed the REF** at (47.8, 50.3)
Connections:
- IC2 pad 16: Net-(IC2-Pad16) -> GND
- IC2 pad 6: Net-(IC2-Pad6) -> GND
- U2 pad 14: /INPUT3 -> Net-(U2-Pad14)
- U2 pad 16: Net-(U2-Pad16) -> /INPUT3
Routing:
- net /BATT_CHECK: track 37.7 -> 42.0 mm
- net /INPUT3: track 16.4 -> 19.3 mm
